Commit message: Add files via upload

File: denso_robot_descriptions/cobotta_description/cobotta.urdf (robot description, URDF)
Before this commit: robot cobotta, 8 links, 7 joints
Joints:
- joint joint_1: limit lower=-2.617994 upper=2.617994 effort=1 velocity=1 -> lower=-2.4 upper=2.4 effort=1 velocity=1
- joint joint_2: limit lower=-1.047198 upper=1.745329 effort=1 velocity=1 -> lower=-0.8 upper=1.6 effort=1 velocity=1
- joint joint_3: limit lower=0.3141593 upper=2.443461 effort=1 velocity=1 -> lower=0.48 upper=2.25 effort=1 velocity=1
- joint joint_4: limit lower=-2.96706 upper=2.96706 effort=1 velocity=1 -> lower=-2.8 upper=2.8 effort=1 velocity=1
- joint joint_5: limit lower=-1.658063 upper=2.356194 effort=1 velocity=1 -> lower=-1.45 upper=2.25 effort=1 velocity=1
- joint joint_6: limit lower=-2.96706 upper=2.96706 effort=1 velocity=1 -> lower=-2.8 upper=2.75 effort=1 velocity=1
